File: Hardware/RCC-motherboard/RCC-motherboard.kicad_sch (KiCad schematic)
At the start: 20 parts, among them J1 1760510000, J2 1760510000, J3 1760510000, J4 1760510000, J5 1760510000, U1 ESP32-DEVKITC-32D, U2 DMG3415U-7, U3 TB6612FNG, U4 TB6612FNG, U5 ZLDO1117G33TA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

Commit message: Designed rough layout for board
Parts:
- removed C2: 10uF, symbol Device:C_Small
- added C10, C12: 0.1uF, Capacitor_SMD:C_0402_1005Metric, symbol Device:C_Small
- added C11, C13, C2, C8, C9: 10uF, Capacitor_SMD:C_1206_3216Metric, symbol Device:C_Polarized_Small
- C1, C3: value 10uF -> 0.1uF; footprint (none) -> Capacitor_SMD:C_0402_1005Metric
- C4, C5: footprint (none) -> Capacitor_SMD:C_1206_3216Metric
- C6, C7: footprint (none) -> CAPMP7343X310N
- R1, R2: footprint (none) -> Resistor_SMD:R_0805_2012Metric
Connections:
- net +3V3: now also C1.1, C10.1, C11.1, C2.1; no longer C3.1
- net +5V: now also C3.1, C12.1, C13.1, C8.1, C9.1; no longer C1.1
- net BIN2_M1: no longer U1.J3-11 (IO17), U3.17 (BIN1)
- net BIN2_M2: no longer U1.J2-10 (IO26), U4.17 (BIN1)
- net GND: now also C10.2, C11.2, C12.2, C13.2, C2.2, C8.2, C9.2
- new net BIN1_M1: U1.J3-11 (IO17), U3.17 (BIN1)
- new net BIN1_M2: U1.J2-10 (IO26), U4.17 (BIN1)
- no-connect marks 0 -> 20
Other:
- note added: "0.1uF CL05A104KA5NNNC"
- note added: "100uF TAJD107K016RNJ"
- note added: "10k resistor: RNCP0805FTD10K0"
- note added: "10uF: TAJA106K016RNJ"
- note added: "PWR FLAGS"
- note added: "TODO: Add capacitors to motor driver design Include the 0.1uF footprint"
- note removed: "TODO: Figure out power distribution to board add power source terminal for motors add power source terminal for board"
- moved on the sheet: J5

Commit message: Finished PCB Layout
Other:
- note added: "Switching Regulator"
- note added: "heatsink requireed"
Changed lines of the file:
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@@
     (effects (font (size 2.27 2.27) (thickness 0.454) bold) (justify left bottom))
+  )
+  (text "heatsink requireed\n" (at 50.8 64.77 0)
+    (effects (font (size 1.27 1.27)) (justify left bottom))
   )
   (text "PWR FLAGS" (at 69.85 105.41 0)
@@
     (effects (font (size 1.27 1.27)) (justify left bottom))
   )
+  (text "Switching Regulator" (at 50.8 62.23 0)
+    (effects (font (size 1.27 1.27)) (justify left bottom))
+  )

Commit message: Produced Gerber and Production files
Parts:
- removed U5: ZLDO1117G33TA, SOT230P700X180-4N, symbol ZLDO1117G33TA:ZLDO1117G33TA
- added H1: MountingHole, MountingHole:MountingHole_3.2mm_M3_ISO7380, symbol Mechanical:MountingHole
- added U5: AZ1117IH-3.3TRG1, SOT230P700X185-4N, symbol AZ1117IH-3.3TRG1:AZ1117IH-3.3TRG1
Connections:
- net +3V3: now also U5.2 (OUTPUT), U5.4 (VOUT)
- net GND: now also U5.1 (GND)
- net Vin: now also U5.3 (INPUT)
Other:
- note added: "Mounting Hole"
- note removed: "TODO: Add capacitors to motor driver design Include the 0.1uF footprint"
- moved on the sheet: C7

Commit message: Created inital Paper Draft
Other:
- company: (none) -> University of Denver
- title: (none) -> BLE Remote Control Board
Changed lines of the file:
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@@
 (kicad_sch (version 20211123) (generator eeschema)
   (paper "A4")
+  (title_block
+    (title "BLE Remote Control Board")
+    (date "2023-04-17")
+    (rev "1")
+    (company "University of Denver")
+  )
   (junction (at 274.32 31.75) (diameter 0) (color 0 0 0 0)
   )
@@
     (effects (font (size 1.27 1.27) (thickness 0.254) bold) (justify left bottom))
   )
-  (text "0.1uF CL05A104KA5NNNC" (at 20.32 139.7 0)
+  (text "0.1uF CL05A104KA5NNNC" (at 20.32 140.97 0)
     (effects (font (size 1.27 1.27)) (justify left bottom))
   )
@@
     (effects (font (size 2.27 2.27) (thickness 0.454) bold) (justify left bottom))
   )
-  (text "100uF TAJD107K016RNJ" (at 20.32 135.89 0)
+  (text "100uF TAJD107K016RNJ" (at 20.32 137.16 0)
     (effects (font (size 1.27 1.27)) (justify left bottom))
   )
@@
     (effects (font (size 2.27 2.27) (thickness 0.454) bold italic) (justify left bottom))
   )
-  (text "10uF: TAJA106K016RNJ\n" (at 20.32 132.08 0)
+  (text "10uF: TAJA106K016RNJ\n" (at 20.32 133.35 0)
     (effects (font (size 1.27 1.27)) (justify left bottom))
   )
@@
     (effects (font (size 1.27 1.27)) (justify left bottom))
   )
-  (text "10k resistor: RNCP0805FTD10K0" (at 20.32 143.51 0)
-    (effects (font (size 1.27 1.27)) (justify left bottom))
-  )
+  (text "10k resistor: RNCP0805FTD10K0" (at 20.32 144.78 0)
+    (effects (font (size 1.27 1.27)) (justify left bottom))
+  )
